File: display/adapter.sch (EAGLE design)
At the start: 17 parts

Commit message: Update
Added partlist and gerber files. Updated some things on board
Parts:
- TM1: value 200 -> 500
Changed lines of the file:
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@@
 <parts>
 <part name="DISPLAY" library="pinhead" library_urn="urn:adsk.eagle:library:325" deviceset="PINHD-1X16" device="" package3d_urn="urn:adsk.eagle:package:22432/2"/>
-<part name="TM1" library="adafruit" library_urn="urn:adsk.eagle:library:420" deviceset="TRIMPOT" device="TC33X" value="200"/>
+<part name="TM1" library="adafruit" library_urn="urn:adsk.eagle:library:420" deviceset="TRIMPOT" device="TC33X" value="500"/>
 <part name="GND1" library="0_HTL_analog" deviceset="GND" device=""/>
 <part name="GND2" library="0_HTL_analog" deviceset="GND" device=""/>
