File: display/adapter.brd (EAGLE design)
At the start: 83.8 x 43.8 mm, 17 parts

Commit message: Update
Added partlist and gerber files. Updated some things on board
Parts:
- TM1: value 200 -> 500
Changed lines of the file:
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@@
 <attribute name="VALUE" x="69.215" y="31.4325" size="1.27" layer="27" rot="R90"/>
 </element>
-<element name="TM1" library="adafruit" library_urn="urn:adsk.eagle:library:420" package="TC33X" value="200" x="52.07" y="12.065" smashed="yes" rot="R180">
+<element name="TM1" library="adafruit" library_urn="urn:adsk.eagle:library:420" package="TC33X" value="500" x="52.07" y="12.065" smashed="yes" rot="R180">
 <attribute name="NAME" x="54.61" y="13.97" size="1.27" layer="25" rot="R270"/>
 <attribute name="VALUE" x="50.8" y="7.62" size="1.27" layer="27"/>

Commit message: Update
Error correction of Display header position.
Parts:
- moved F1 4.00 mm to (41.7, 12.1)
- moved TM1 4.00 mm to (48.1, 12.1)
- moved TM2 4.00 mm to (37.9, 12.1)
- moved DISPLAY 3.90 mm to (29.1, 3.75)
Routing:
- net DB7: track 39.0 -> 43.4 mm
- net DB6: track 35.4 -> 39.3 mm
- net RS: track 47.2 -> 43.6 mm
- net E: track 46.9 -> 43.4 mm
- net DB5: track 38.0 -> 41.2 mm
- net DB4: track 34.4 -> 37.1 mm
- net N$4: track 52.6 -> 54.7 mm
- net +3V3: vias 3 -> 4
