File: display/adapter.brd (EAGLE design)
At the start: 83.8 x 43.8 mm, 17 parts

Commit message: Update
Added a new design (controller) and corrected again some things in the display project...
Parts:
- moved F1 0.81 mm to (42.6, 12.2)
- moved TM1 0.81 mm to (48.1, 12.2)
- moved TM2 0.81 mm to (37.9, 12.2)
- moved DISPLAY 0.80 mm to (29.1, 3.75)
